File: arduino-nano-connectors.kicad_sch (KiCad schematic)
At the start: 2 parts, among them J65 Conn_01x15, J66 Conn_01x15

Commit message: removing extra files
Changed lines of the file:
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@@
 		)
 		(property "Value" "Conn_01x15"
-			(at 153.5684 90.5764 90)
+			(at 154.432 90.678 90)
 			(effects
 				(font
