File: chess.kicad_sch (KiCad schematic)
At the start: 0 parts

Commit message: removing extra files
Changed lines of the file:
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@@
 	(wire
 		(pts
-			(xy 39.37 27.94) (xy 41.91 27.94)
+			(xy 39.37 26.67) (xy 41.91 26.67)
 		)
 		(stroke
@@
 	(wire
 		(pts
-			(xy 41.91 27.94) (xy 41.91 35.56)
+			(xy 41.91 26.67) (xy 41.91 35.56)
 		)
 		(stroke
@@
 	)
 	(sheet
-		(at 26.67 25.4)
+		(at 26.67 24.13)
 		(size 12.7 3.81)
 		(fields_autoplaced yes)
@@
 		)
 		(property "Sheetname" "row1"
-			(at 26.67 24.6884 0)
+			(at 26.67 23.4184 0)
 			(effects
 				(font
@@
 		)
 		(property "Sheetfile" "row.kicad_sch"
-			(at 26.67 29.7946 0)
+			(at 26.67 28.5246 0)
 			(effects
 				(font
@@
 		)
 		(pin "IN" input
-			(at 26.67 27.94 180)
+			(at 26.67 26.67 180)
 			(effects
 				(font
@@
 		)
 		(pin "OUT" output
-			(at 39.37 27.94 0)
-			(effects
-				(font
+			(at 39.37 26.67 0)
+			(effects
+				(font
