File: input.kicad_sch (KiCad schematic)
At the start: 3 parts, among them J1 PINHD_1x1_Male

Commit message: removing extra files
Changed lines of the file:
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@@
 	(wire
 		(pts
-			(xy 38.1 31.75) (xy 38.1 27.94)
+			(xy 38.1 31.75) (xy 38.1 29.21)
 		)
 		(stroke
@@
 	(wire
 		(pts
-			(xy 38.1 27.94) (xy 48.26 27.94)
+			(xy 38.1 29.21) (xy 48.26 29.21)
 		)
 		(stroke
@@
 	(symbol
 		(lib_id "power:GND")
-		(at 48.26 27.94 0)
+		(at 48.26 29.21 0)
 		(unit 1)
 		(exclude_from_sim no)
@@
 		(on_board yes)
 		(dnp no)
-		(fields_autoplaced yes)
 		(property "Reference" "#PWR0101"
-			(at 48.26 34.29 0)
+			(at 48.26 35.56 0)
 			(effects
 				(font
@@
 		)
 		(property "Value" "GND"
-			(at 48.26 33.02 0)
+			(at 48.26 34.29 0)
 			(effects
 				(font
@@
 		)
 		(property "Footprint" ""
-			(at 48.26 27.94 0)
+			(at 48.26 29.21 0)
 			(effects
 				(font
@@
 		)
 		(property "Datasheet" ""
-			(at 48.26 27.94 0)
+			(at 48.26 29.21 0)
 			(effects
 				(font
@@
 		)
 		(property "Description" "Power symbol creates a global label with name \"GND\" , ground"
-			(at 48.26 27.94 0)
+			(at 48.26 29.21 0)
 			(effects
 				(font
