File: inputshield.kicad_pcb (KiCad board)
At the start: 2 copper layers, 200 x 108 mm, 211 parts, among them J1 PINHD_1x1_Male, J10 PINHD_1x1_Male, J11 PINHD_1x1_Male, J12 PINHD_1x1_Male, J13 PINHD_1x1_Male, J14 PINHD_1x1_Male, J15 PINHD_1x1_Male, J16 PINHD_1x1_Male, J17 PINHD_1x1_Male, J18 PINHD_1x1_Male, J19 PINHD_1x1_Male, J2 PINHD_1x1_Male, J20 PINHD_1x1_Male, J21 PINHD_1x1_Male, J22 PINHD_1x1_Male, J23 PINHD_1x1_Male, J24 PINHD_1x1_Male, J25 PINHD_1x1_Male, J26 PINHD_1x1_Male, J27 PINHD_1x1_Male, J28 PINHD_1x1_Male, J29 PINHD_1x1_Male, J3 PINHD_1x1_Male, J30 PINHD_1x1_Male, J31 PINHD_1x1_Male, J32 PINHD_1x1_Male, J33 PINHD_1x1_Male, J34 PINHD_1x1_Male, J35 PINHD_1x1_Male, J36 PINHD_1x1_Male, J37 PINHD_1x1_Male, J38 PINHD_1x1_Male, J39 PINHD_1x1_Male, J4 PINHD_1x1_Male, J40 PINHD_1x1_Male, J41 PINHD_1x1_Male, J42 PINHD_1x1_Male, J43 PINHD_1x1_Male, J44 PINHD_1x1_Male, J45 PINHD_1x1_Male, J46 PINHD_1x1_Male, J47 PINHD_1x1_Male, J48 PINHD_1x1_Male, J49 PINHD_1x1_Male, J5 PINHD_1x1_Male, J50 PINHD_1x1_Male, J51 PINHD_1x1_Male, J52 PINHD_1x1_Male, J53 PINHD_1x1_Male, J54 PINHD_1x1_Male, J55 PINHD_1x1_Male, J56 PINHD_1x1_Male, J57 PINHD_1x1_Male, J58 PINHD_1x1_Male, J59 PINHD_1x1_Male, J6 PINHD_1x1_Male, J60 PINHD_1x1_Male, J61 PINHD_1x1_Male, J62 PINHD_1x1_Male, J63 PINHD_1x1_Male, J64 PINHD_1x1_Male, J65 Conn_01x15, J66 Conn_01x15, J67 Conn_02x15_Counter_Clockwise_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, J7 PINHD_1x1_Male, J8 PINHD_1x1_Male, J9 PINHD_1x1_Male, U1 SN74HC165N, U2 SN74HC165N, U3 SN74HC165N, U4 SN74HC165N, U5 SN74HC165N, U6 SN74HC165N, U7 SN74HC165N, U8 SN74HC165N

Commit message: removing extra files
Parts:
- moved C3 20.8 mm to (140.2, 60.8)
- moved C4 20.8 mm to (169.7, 60.8)
- moved C7 20.8 mm to (140.2, 107.2)
- moved C8 20.8 mm to (169.7, 106.8)
- moved J17 20.8 mm to (134.7, 51.5)
- moved J18 20.8 mm to (130.7, 51.5)
- moved J23 20.8 mm to (131.2, 69.8)
- moved J24 20.8 mm to (135.2, 69.8)
- moved J25 20.8 mm to (164.7, 51.5)
- moved J26 20.8 mm to (160.7, 51.5)
- moved J27 20.8 mm to (156.7, 51.5)
- moved J28 20.8 mm to (152.7, 51.5)
- moved J29 20.8 mm to (152.7, 69.8)
- moved J30 20.8 mm to (156.7, 69.8)
- moved J31 20.8 mm to (160.7, 69.8)
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