File: inputshield.kicad_sch (KiCad schematic)
At the start: 1 part, among them J67 Conn_02x15_Counter_Clockwise_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

Commit message: removing extra files
Changed lines of the file:
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@@
 	(wire
 		(pts
-			(xy 99.06 60.96) (xy 104.14 60.96)
+			(xy 99.06 59.69) (xy 104.14 59.69)
 		)
 		(stroke
@@
 	(wire
 		(pts
-			(xy 104.14 60.96) (xy 104.14 76.2)
+			(xy 104.14 59.69) (xy 104.14 76.2)
 		)
 		(stroke
@@
 	)
 	(sheet
-		(at 86.36 59.69)
+		(at 86.36 58.42)
 		(size 12.7 3.81)
 		(fields_autoplaced yes)
@@
 		)
 		(property "Sheetname" "chess"
-			(at 86.36 58.9784 0)
+			(at 86.36 57.7084 0)
 			(effects
 				(font
@@
 		)
 		(property "Sheetfile" "chess.kicad_sch"
-			(at 86.36 64.0846 0)
+			(at 86.36 62.8146 0)
 			(effects
 				(font
@@
 		)
 		(pin "OUT" output
-			(at 99.06 60.96 0)
-			(effects
-				(font
+			(at 99.06 59.69 0)
+			(effects
+				(font
