File: row.kicad_sch (KiCad schematic)
At the start: 2 parts, among them U1 SN74HC165N

Commit message: removing extra files
Changed lines of the file:
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@@
 	(wire
 		(pts
-			(xy 99.06 88.9) (xy 55.88 88.9)
+			(xy 99.06 88.9) (xy 54.61 88.9)
 		)
 		(stroke
@@
 	(wire
 		(pts
-			(xy 55.88 88.9) (xy 55.88 118.11)
+			(xy 54.61 88.9) (xy 54.61 118.11)
 		)
 		(stroke
@@
 	)
 	(sheet
-		(at 53.34 118.11)
+		(at 52.07 118.11)
 		(size 12.7 3.81)
 		(fields_autoplaced yes)
@@
 		)
 		(property "Sheetname" "input1"
-			(at 52.6284 121.92 90)
+			(at 51.3584 121.92 90)
 			(effects
 				(font
@@
 		)
 		(property "Sheetfile" "input.kicad_sch"
-			(at 66.6246 121.92 90)
+			(at 65.3546 121.92 90)
 			(effects
 				(font
@@
 		)
 		(pin "I1" output
-			(at 55.88 118.11 90)
-			(effects
-				(font
+			(at 54.61 118.11 90)
+			(effects
+				(font
